File: Project 1.kicad_pcb (KiCad board)
At the start: 2 copper layers, 14 parts, among them J1 DB9_Female, J2 Barrel_Jack, P1 RFID-RC522-MODULE, SW1 SW_DPDT_x2, U1 PIC16F1512-ISP, U2 PIC16F1512-ISP, U3 PIC16F1512-ISP, U4 ADG419BN, U5 TM1637, U6 TM1637

Commit message: Nieuwe tekening begin nieuw schema
Nieuwe tekening begin nieuw schema
Parts:
- removed U2: PIC16F1512-ISP, Package_DIP:DIP-28_W7.62mm
- removed U3: PIC16F1512-ISP, Package_DIP:DIP-28_W7.62mm_Socket
- P1: footprint Connector_PinHeader_1.27mm:PinHeader_1x08_P1.27mm_Vertical -> Connector_PinSocket_2.54mm:PinSocket_1x08_P2.54mm_Vertical
- moved U5 89.3 mm to (12.7, 48.8)
- moved SW1 87.0 mm to (96.5, 100.1), turned to 0 degrees
- moved U6 58.2 mm to (59.4, 48.8)
- moved J2 52.4 mm to (113.3, 71.6), turned to 180 degrees
- moved R1 51.7 mm to (116.3, 40.1)
- moved R3 50.6 mm to (116.3, 42.2)
- moved D1 49.9 mm to (109.7, 41.7)
- moved R2 47.5 mm to (116.3, 43.7)
- moved J1 45.8 mm to (99.7, 85.8), turned to -90 degrees
- moved U1 44.3 mm to (77.0, 65.8)
- moved U4 29.3 mm to (110.7, 92.5), turned to 90 degrees
- moved P1 10.1 mm to (12.7, 79.0)
Connections:
- D1 pad 1: Net-(U3-Pad28) -> Net-(U1-Pad28)
- D1 pad 2: Net-(U3-Pad27) -> Net-(U1-Pad27)
- D1 pad 3: Net-(U3-Pad26) -> Net-(U1-Pad26)
- J2 pad 1: Net-(SW1-Pad3) -> Net-(J2-Pad1)
- R1 pad 2: unconnected-(R1-Pad2) -> GNDREF
- R2 pad 2: unconnected-(R2-Pad2) -> GNDREF
- R3 pad 2: unconnected-(R3-Pad2) -> GNDREF
- SW1 pad 2: Net-(U1-Pad20) -> Net-(J2-Pad1)
- SW1 pad 3: Net-(SW1-Pad3) -> +5V
- U1 pad 10: Net-(U3-Pad9) -> unconnected-(U1-Pad10)
- U1 pad 15: Net-(U3-Pad15) -> unconnected-(U1-Pad15)
- U1 pad 16: unconnected-(U1-Pad16) -> Net-(U1-Pad16)
- U1 pad 20: Net-(U1-Pad20) -> +5V
- U1 pad 25: unconnected-(U1-Pad25) -> Net-(U1-Pad25)
- U1 pad 26: unconnected-(U1-Pad26) -> Net-(U1-Pad26)
- U1 pad 27: unconnected-(U1-Pad27) -> Net-(U1-Pad27)
- U1 pad 28: unconnected-(U1-Pad28) -> Net-(U1-Pad28)
- U4 pad 1: Net-(U3-Pad16) -> Net-(U1-Pad16)
- U4 pad 6: Net-(U4-Pad6) -> Net-(U1-Pad25)
- U5 pad 4: Net-(U1-Pad20) -> unconnected-(U5-Pad4)
- U6 pad 4: Net-(U1-Pad20) -> +5V
Other:
- board outline added: 112.3 x 67.1 mm
